File: STM32MP1_TestBoard/STM32MP1_TestBoard.sch (KiCad schematic (older format))
At the start: 16 parts, among them J10 Conn_01x12, J3 Conn_01x16, J4 Conn_01x16, J5 Conn_01x16, J6 Conn_01x16, J7 Conn_02x03_Odd_Even, J8 Conn_01x16, J9 Conn_01x06, U1 STM32MP157xAB

Commit message: updated bom, readme
Parts:
- removed U1: STM32MP157xAB, STM32MP151_LFBGA:BGA-361_19x19_16.0x16.0mm, symbol STM32MP151:STM32MP151xAB
- added J15: Conn_01x06, Connector_PinHeader_2.54mm:PinHeader_1x06_P2.54mm_Vertical, symbol Connector_Generic:Conn_01x06
- added U1: STM32MP157xAB, STM32MP151_LFBGA:BGA-361_19x19_16.0x16.0mm, symbol STM32MP15x:STM32MP157xAB
- J10: footprint (none) -> Connector_PinHeader_2.54mm:PinHeader_1x12_P2.54mm_Vertical
- J7: footprint (none) -> Connector_PinHeader_2.54mm:PinHeader_2x03_P2.54mm_Vertical
- J9: footprint (none) -> Connector_PinHeader_2.54mm:PinHeader_1x06_P2.54mm_Vertical
- gave numbers to parts that had none: 4
Connections:
- wire segments 167 -> 173
- no-connect marks 9 -> 3
Changed lines of the file:
@@
 $EndDescr
-$Comp
-L STM32MP151:STM32MP151xAB U1
-U 1 1 5FA92710
-P 9650 9400
-F 0 "U1" H 9700 11565 50  0000 C CNN
-F 1 "STM32MP157xAB" H 9700 11474 50  0000 C CNN
-F 2 "STM32MP151_LFBGA:BGA-361_19x19_16.0x16.0mm" H 9550 14650 50  0001 C CNN
-F 3 "https://www.st.com/resource/en/datasheet/stm32mp157d.pdf" H 9900 12550 50  0001 C CNN
-F 4 "STMicroelectronics" H 9650 9400 50  0001 C CNN "Mfr"
-F 5 "STM32MP151DAB" H 9650 9400 50  0001 C CNN "PartNo"
-	1    9650 9400
-	1    0    0    -1
-$EndComp
-$Comp
-L STM32MP151:STM32MP151xAB U1
-U 2 1 5FA99B00
-P 17725 9300
-F 0 "U1" H 17725 10865 50  0000 C CNN
-F 1 "STM32MP157xAB" H 17725 10774 50  0000 C CNN
-F 2 "STM32MP151_LFBGA:BGA-361_19x19_16.0x16.0mm" H 17625 14550 50  0001 C CNN
-F 3 "https://www.st.com/resource/en/datasheet/stm32mp157d.pdf" H 17975 12450 50  0001 C CNN
-F 4 "STMicroelectronics" H 17725 9300 50  0001 C CNN "Mfr"
-F 5 "STM32MP151DAB" H 17725 9300 50  0001 C CNN "PartNo"
-	2    17725 9300
-	1    0    0    -1
-$EndComp
 $Comp
 L power:+3.3V #PWR012
@@
 F 2 "Connector_PinHeader_2.54mm:PinHeader_1x16_P2.54mm_Vertical" H 7025 8200 50  0001 C CNN
 F 3 "~" H 7025 8200 50  0001 C CNN
+F 4 "~" H 7025 8200 50  0001 C CNN "Mfr"
+F 5 "~" H 7025 8200 50  0001 C CNN "PartNo"
 	1    7025 8200
 	-1   0    0    -1
@@
 F 2 "Connector_PinHeader_2.54mm:PinHeader_1x16_P2.54mm_Vertical" H 7025 9950 50  0001 C CNN
 F 3 "~" H 7025 9950 50  0001 C CNN
+F 4 "~" H 7025 9950 50  0001 C CNN "Mfr"
+F 5 "~" H 7025 9950 50  0001 C CNN "PartNo"
 	1    7025 9950
 	-1   0    0    -1
@@
 F 2 "Connector_PinHeader_2.54mm:PinHeader_1x16_P2.54mm_Vertical" H 12375 8200 50  0001 C CNN
 F 3 "~" H 12375 8200 50  0001 C CNN
+F 4 "~" H 12375 8200 50  0001 C CNN "Mfr"
+F 5 "~" H 12375 8200 50  0001 C CNN "PartNo"
 	1    12375 8200
 	1    0    0    -1
@@
 F 2 "Connector_PinHeader_2.54mm:PinHeader_1x16_P2.54mm_Vertical" H 12375 9950 50  0001 C CNN
 F 3 "~" H 12375 9950 50  0001 C CNN
+F 4 "~" H 12375 9950 50  0001 C CNN "Mfr"
+F 5 "~" H 12375 9950 50  0001 C CNN "PartNo"
 	1    12375 9950
 	1    0    0    -1
@@
 F 2 "Connector_PinHeader_2.54mm:PinHeader_1x16_P2.54mm_Vertical" H 15050 8700 50  0001 C CNN
 F 3 "~" H 15050 8700 50  0001 C CNN
+F 4 "~" H 15050 8700 50  0001 C CNN "Mfr"
+F 5 "~" H 15050 8700 50  0001 C CNN "PartNo"
 	1    15050 8700
 	-1   0    0    -1
@@
 Wire Wire Line
 	15250 9500 16825 9500
-NoConn ~ 18625 9300
-NoConn ~ 18625 9400
-NoConn ~ 18625 9500
-NoConn ~ 18625 9600
-NoConn ~ 18625 9700
-NoConn ~ 18625 9800
 $Comp
 L Connector_Generic:Conn_01x06 J9
@@
 F 0 "J9" H 15425 9925 50  0000 C CNN
 F 1 "Conn_01x06" H 15425 9825 50  0000 C CNN
-F 2 "" H 15050 9900 50  0001 C CNN
+F 2 "Connector_PinHeader_2.54mm:PinHeader_1x06_P2.54mm_Vertical" H 15050 9900 50  0001 C CNN
 F 3 "~" H 15050 9900 50  0001 C CNN
+F 4 "~" H 15050 9900 50  0001 C CNN "Mfr"
+F 5 "~" H 15050 9900 50  0001 C CNN "PartNo"
 	1    15050 9900
 	-1   0    0    -1
@@
 F 0 "J10" H 19930 8492 50  0000 L CNN
 F 1 "Conn_01x12" H 19930 8401 50  0000 L CNN
-F 2 "" H 19850 8500 50  0001 C CNN
+F 2 "Connector_PinHeader_2.54mm:PinHeader_1x12_P2.54mm_Vertical" H 19850 8500 50  0001 C CNN
 F 3 "~" H 19850 8500 50  0001 C CNN
+F 4 "~" H 19850 8500 50  0001 C CNN "Mfr"
+F 5 "~" H 19850 8500 50  0001 C CNN "PartNo"
 	1    19850 8500
 	1    0    0    -1
@@
 F 0 "J7" H 15050 10300 50  0000 C CNN
 F 1 "Conn_02x03_Odd_Even" H 15075 10225 50  0000 C CNN
-F 2 "" H 15000 10500 50  0001 C CNN
+F 2 "Connector_PinHeader_2.54mm:PinHeader_2x03_P2.54mm_Vertical" H 15000 10500 50  0001 C CNN
 F 3 "~" H 15000 10500 50  0001 C CNN
+F 4 "~" H 15000 10500 50  0001 C CNN "Mfr"
+F 5 "~" H 15000 10500 50  0001 C CNN "PartNo"
 	1    15000 10500
 	1    0    0    -1
@@
 F 2 "Resistor_SMD:R_0402_1005Metric_Pad0.72x0.64mm_HandSolder" V 15880 11300 50  0001 C CNN
 F 3 "~" H 15950 11300 50  0001 C CNN
+F 4 "~" H 15950 11300 50  0001 C CNN "Mfr"
+F 5 "~" H 15950 11300 50  0001 C CNN "PartNo"
 	1    15950 11300
 	1    0    0    -1
@@
 F 2 "Resistor_SMD:R_0402_1005Metric_Pad0.72x0.64mm_HandSolder" V 16180 11300 50  0001 C CNN
 F 3 "~" H 16250 11300 50  0001 C CNN
+F 4 "~" H 16250 11300 50  0001 C CNN "Mfr"
+F 5 "~" H 16250 11300 50  0001 C CNN "PartNo"
 	1    16250 11300
 	1    0    0    -1
@@
 F 2 "Resistor_SMD:R_0402_1005Metric_Pad0.72x0.64mm_HandSolder" V 16480 11300 50  0001 C CNN
 F 3 "~" H 16550 11300 50  0001 C CNN
+F 4 "~" H 16550 11300 50  0001 C CNN "Mfr"
+F 5 "~" H 16550 11300 50  0001 C CNN "PartNo"
 	1    16550 11300
 	1    0    0    -1
@@
 NoConn ~ 8800 11000
 $Comp
-L Device:R R?
+L Device:R R5
 U 1 1 6083D116
 P 8150 11725
-F 0 "R?" H 8275 11675 50  0000 C CNN
+F 0 "R5" H 8275 11675 50  0000 C CNN
 F 1 "3K" H 8275 11775 50  0000 C CNN
 F 2 "Resistor_SMD:R_0402_1005Metric_Pad0.72x0.64mm_HandSolder" V 8080 11725 50  0001 C CNN
 F 3 "~" H 8150 11725 50  0001 C CNN
+F 4 "~" H 8150 11725 50  0001 C CNN "Mfr"
+F 5 "~" H 8150 11725 50  0001 C CNN "PartNo"
 	1    8150 11725
 	-1   0    0    1
@@
 	8150 11875 8150 12025
 $Comp
-L power:GNDS #PWR?
+L power:GNDS #PWR0101
 U 1 1 6084EC4C
 P 8150 12025
-F 0 "#PWR?" H 8150 11775 50  0001 C CNN
+F 0 "#PWR0101" H 8150 11775 50  0001 C CNN
 F 1 "GNDS" H 8155 11852 50  0000 C CNN
 F 2 "" H 8150 12025 50  0001 C CNN
@@
 	19050 10600 19050 10925
 $Comp
-L power:GNDS #PWR?
+L power:GNDS #PWR0102
 U 1 1 60E59490
 P 19050 10925
-F 0 "#PWR?" H 19050 10675 50  0001 C CNN
+F 0 "#PWR0102" H 19050 10675 50  0001 C CNN
 F 1 "GNDS" H 19055 10752 50  0000 C CNN
 F 2 "" H 19050 10925 50  0001 C CNN
@@
 	19650 10500 19650 10575
 $Comp
-L Device:C C?
+L Device:C C39
 U 1 1 60E63E33
 P 19650 10725
-F 0 "C?" H 19765 10771 50  0000 L CNN
+F 0 "C39" H 19765 10771 50  0000 L CNN
 F 1 "10nF" H 19765 10680 50  0000 L CNN
 F 2 "Capacitor_SMD:C_0402_1005Metric_Pad0.74x0.62mm_HandSolder" H 19688 10575 50  0001 C CNN
 F 3 "~" H 19650 10725 50  0001 C CNN
+F 4 "~" H 19650 10725 50  0001 C CNN "Mfr"
+F 5 "~" H 19650 10725 50  0001 C CNN "PartNo"
 	1    19650 10725
 	1    0    0    -1
@@
 	19650 10875 19650 10925
 $Comp
-L power:GNDS #PWR?
+L power:GNDS #PWR0103
 U 1 1 60E6488D
 P 19650 10925
-F 0 "#PWR?" H 19650 10675 50  0001 C CNN
+F 0 "#PWR0103" H 19650 10675 50  0001 C CNN
 F 1 "GNDS" H 19655 10752 50  0000 C CNN
 F 2 "" H 19650 10925 50  0001 C CNN
@@
 	20300 10400 20300 10300
 $Comp
-L power:+3.3V #PWR?
+L power:+3.3V #PWR0104
 U 1 1 60E7A234
-P 20300 9950
-F 0 "#PWR?" H 20300 9800 50  0001 C CNN
-F 1 "+3.3V" H 20315 10123 50  0000 C CNN
-F 2 "" H 20300 9950 50  0001 C CNN
-F 3 "" H 20300 9950 50  0001 C CNN
-	1    20300 9950
+P 20300 10100
+F 0 "#PWR0104" H 20300 9950 50  0001 C CNN
+F 1 "+3.3V" H 20315 10273 50  0000 C CNN
+F 2 "" H 20300 10100 50  0001 C CNN
+F 3 "" H 20300 10100 50  0001 C CNN
+	1    20300 10100
 	1    0    0    -1
 $EndComp
@@
 Connection ~ 20300 10300
 Wire Wire Line
-	20300 10300 20300 9950
+	20300 10300 20300 10100
 Wire Wire Line
 	18625 10200 19350 10200
@@
 P 19350 10200
 AR Path="/60386EBB/60EAB252" Ref="TP?"  Part="1"
-AR Path="/60EAB252" Ref="TP?"  Part="1"
-F 0 "TP?" V 19350 10388 50  0000 L CNN
+AR Path="/60EAB252" Ref="TP4"  Part="1"
+F 0 "TP4" V 19350 10388 50  0000 L CNN
 F 1 "~" V 19395 10388 50  0000 L CNN
 F 2 "TestPoint:TestPoint_Pad_D1.0mm" H 19550 10200 50  0001 C CNN
 F 3 "~" H 19550 10200 50  0001 C CNN
+F 4 "~" H 19350 10200 50  0001 C CNN "Mfr"
+F 5 "~" H 19350 10200 50  0001 C CNN "PartNo"
 	1    19350 10200
 	0    1    1    0
@@
 P 19475 10500
 AR Path="/60386EBB/60EB52ED" Ref="TP?"  Part="1"
-AR Path="/60EB52ED" Ref="TP?"  Part="1"
-F 0 "TP?" V 19475 10688 50  0000 L CNN
+AR Path="/60EB52ED" Ref="TP5"  Part="1"
+F 0 "TP5" V 19475 10688 50  0000 L CNN
 F 1 "~" V 19520 10688 50  0000 L CNN
 F 2 "TestPoint:TestPoint_Pad_D1.0mm" H 19675 10500 50  0001 C CNN
 F 3 "~" H 19675 10500 50  0001 C CNN
+F 4 "~" H 19475 10500 50  0001 C CNN "Mfr"
+F 5 "~" H 19475 10500 50  0001 C CNN "PartNo"
 	1    19475 10500
 	-1   0    0    1
@@
 Wire Wire Line
 	8800 11400 4600 11400
+$Comp
+L STM32MP15x:STM32MP157xAB U1
+U 1 1 602257F2
+P 9650 9400
+F 0 "U1" H 9700 11565 50  0000 C CNN
+F 1 "STM32MP157xAB" H 9700 11474 50  0000 C CNN
+F 2 "STM32MP151_LFBGA:BGA-361_19x19_16.0x16.0mm" H 9500 11300 50  0001 C CNN
+F 3 "https://www.st.com/resource/en/datasheet/stm32mp157f.pdf" H 9950 9900 50  0001 C CNN
+F 4 "STMicroelectronics" H 9650 9400 50  0001 C CNN "Mfr"
+F 5 "STM32MP157FAB" H 9650 9400 50  0001 C CNN "PartNo"
+	1    9650 9400
+	1    0    0    -1
+$EndComp
+$Comp
+L STM32MP15x:STM32MP157xAB U1
+U 2 1 60232850
+P 17725 9300
+F 0 "U1" H 17725 10865 50  0000 C CNN
+F 1 "STM32MP157xAB" H 17725 10774 50  0000 C CNN
+F 2 "STM32MP151_LFBGA:BGA-361_19x19_16.0x16.0mm" H 17575 11200 50  0001 C CNN
+F 3 "https://www.st.com/resource/en/datasheet/stm32mp157f.pdf" H 18025 9800 50  0001 C CNN
+F 4 "STMicroelectronics" H 17725 9300 50  0001 C CNN "Mfr"
+F 5 "STM32MP157FAB" H 17725 9300 50  0001 C CNN "PartNo"
+	2    17725 9300
+	1    0    0    -1
+$EndComp
+$Comp
+L Connector_Generic:Conn_01x06 J15
+U 1 1 60240A56
+P 19850 9500
+F 0 "J15" H 19975 9525 50  0000 C CNN
+F 1 "Conn_01x06" H 20150 9425 50  0000 C CNN
+F 2 "Connector_PinHeader_2.54mm:PinHeader_1x06_P2.54mm_Vertical" H 19850 9500 50  0001 C CNN
+F 3 "~" H 19850 9500 50  0001 C CNN
+F 4 "~" H 19850 9500 50  0001 C CNN "Mfr"
+F 5 "~" H 19850 9500 50  0001 C CNN "PartNo"
+	1    19850 9500
+	1    0    0    -1
+$EndComp
+Wire Wire Line
+	19650 9300 18625 9300
+Wire Wire Line
+	18625 9400 19650 9400
+Wire Wire Line
+	18625 9500 19650 9500
+Wire Wire Line
+	19650 9600 18625 9600
+Wire Wire Line
+	18625 9700 19650 9700
+Wire Wire Line
+	19650 9800 18625 9800
 $EndSCHEMATC

Commit message: minor schema updates
Parts:
- added C5: 10nF, Capacitor_SMD:C_0402_1005Metric_Pad0.74x0.62mm_HandSolder, symbol Device:C
- added D1: LED, LED_SMD:LED_0805_2012Metric_Pad1.15x1.40mm_HandSolder, symbol Device:LED
- added JP1: Jumper_NO_Small, Jumper:SolderJumper-2_P1.3mm_Open_RoundedPad1.0x1.5mm, symbol Device:Jumper_NO_Small
- added R1: 680R, Resistor_SMD:R_0402_1005Metric_Pad0.72x0.64mm_HandSolder, symbol Device:R
- added SW1: SW_SPST, Button_Switch_SMD:Panasonic_EVQPUK_EVQPUB, symbol Switch:SW_SPST
Connections:
- net labels added: +3V3, BOOT_STATUS
- wire segments 173 -> 181
Other:
- note added: "BOOT MODE BOOT2 BOOT1. BOOT1\n———————————————————————————————\nSDCard 1 0 1\nForced UART/USB. 0 0 0\nDisable Flash boot 1 0 0"
- note added: "On silicon Rev.B, recommended \nconnection when there is no \nVDDCORE power cycle on NRST \n(done by default with STPMIC1)"
- note removed: "BOOT MODE BOOT2 BOOT1. BOOT1\n———————————————————————\nSDCard 1 0 1\nForced UART/USB. 0 0 0\nReserved 1 0 0"
- moved on the sheet: R7, R8, R9

Commit message: updated schematic design
Parts:
- removed C39, C5: 10nF, Capacitor_SMD:C_0402_1005Metric_Pad0.74x0.62mm_HandSolder, symbol Device:C
- removed D1: LED, LED_SMD:LED_0805_2012Metric_Pad1.15x1.40mm_HandSolder, symbol Device:LED
- removed J10: Conn_01x12, Connector_PinHeader_2.54mm:PinHeader_1x12_P2.54mm_Vertical, symbol Connector_Generic:Conn_01x12
- removed J15, J9: Conn_01x06, Connector_PinHeader_2.54mm:PinHeader_1x06_P2.54mm_Vertical, symbol Connector_Generic:Conn_01x06
- removed J3, J4, J5, J6, J8: Conn_01x16, Connector_PinHeader_2.54mm:PinHeader_1x16_P2.54mm_Vertical, symbol Connector_Generic:Conn_01x16
- removed J7: Conn_02x03_Odd_Even, Connector_PinHeader_2.54mm:PinHeader_2x03_P2.54mm_Vertical, symbol Connector_Generic:Conn_02x03_Odd_Even
- removed JP1: Jumper_NO_Small, Jumper:SolderJumper-2_P1.3mm_Open_RoundedPad1.0x1.5mm, symbol Device:Jumper_NO_Small
- removed R1: 680R, Resistor_SMD:R_0402_1005Metric_Pad0.72x0.64mm_HandSolder, symbol Device:R
- removed R5: 3K, Resistor_SMD:R_0402_1005Metric_Pad0.72x0.64mm_HandSolder, symbol Device:R
- removed R7, R8, R9: 1K, Resistor_SMD:R_0402_1005Metric_Pad0.72x0.64mm_HandSolder, symbol Device:R
- removed SW1: SW_SPST, Button_Switch_SMD:Panasonic_EVQPUK_EVQPUB, symbol Switch:SW_SPST
- removed TP4, TP5: ~, TestPoint:TestPoint_Pad_D1.0mm, symbol Connector:TestPoint
- removed U1: STM32MP157xAB, STM32MP151_LFBGA:BGA-361_19x19_16.0x16.0mm, symbol STM32MP15x:STM32MP157xAB
Connections:
- net labels removed: +1V35, +3.3V, +3V3, BOOT_STATUS, GNDS, NRST, PWR_CTRL_ON, SDMMC1_CK, SDMMC1_CMD, SDMMC1_D0, SDMMC1_D1, SDMMC1_D2, SDMMC1_D3, SDMMC2_CK, SDMMC2_CMD, SDMMC2_D0, SDMMC2_D1, SDMMC2_D2, SDMMC2_D3, SWCLK, SWDIO, SWO
- wire segments 181 -> 16
- no-connect marks 3 -> 0
Other:
- note added: "<- ENABLE 3V3_USB"
- note added: "<- ENABLE VDDCORE"
- note added: "PWR_OUT -->"
- note removed: "BOOT MODE BOOT2 BOOT1. BOOT1\n———————————————————————————————\nSDCard 1 0 1\nForced UART/USB. 0 0 0\nDisable Flash boot 1 0 0"
- note removed: "On silicon Rev.B, recommended \nconnection when there is no \nVDDCORE power cycle on NRST \n(done by default with STPMIC1)"

Commit message: layout update
backup. work in progress
Changed lines of the file:
@@
 F4 "PWR_ON" I L 9350 4650 50
 F5 "1.35V_VDDCORE" I L 9350 4500 50
-F6 "3.3v_VDD" I L 9350 5675 50
+F6 "3.3V_VDD" I L 9350 5675 50
 $EndSheet
 Wire Wire Line
@@
 F1 "PSU.sch" 50
 F2 "3V3_USB" I R 6050 5025 50
-F4 "1.35V_VDDCORE" I R 6050 4075 50
-F5 "3.3V_VDD" I R 6050 5675 50
-F6 "1V8_DETECT" I R 6050 5225 50
-F7 "PWR_ON" I R 6050 4650 50
+F3 "1.35V_VDDCORE" I R 6050 4075 50
+F4 "3.3V_VDD" I R 6050 5675 50
+F5 "1V8_DETECT" I R 6050 5225 50
+F6 "PWR_ON" I R 6050 4650 50
 $EndSheet
 Wire Wire Line

Commit message: updated RevA draft
- added silkscreen
Other:
- note removed: "<- ENABLE VDDCORE"
Changed lines of the file:
@@
 F2 "3V3_USB" I L 9350 5025 50
 F3 "1V8_DETECT" I L 9350 5225 50
-F4 "PWR_ON" I L 9350 4650 50
 F5 "1.35V_VDDCORE" I L 9350 4500 50
 F6 "3.3V_VDD" I L 9350 5675 50
@@
 F4 "3.3V_VDD" I R 6050 5675 50
 F5 "1V8_DETECT" I R 6050 5225 50
-F6 "PWR_ON" I R 6050 4650 50
 $EndSheet
-Wire Wire Line
-	9350 5025 6050 5025
 $Sheet
 S 4500 6650 1525 675
@@
 F2 "3.3V_VDD" I R 6025 6950 50
 $EndSheet
-Wire Wire Line
-	6050 4650 9350 4650
 $Sheet
 S 9350 6625 1800 700
@@
 	7375 4500 7375 4075
 Connection ~ 7375 4075
-Text Notes 6225 4650 0    50   ~ 0
-<- ENABLE VDDCORE
 Text Notes 6200 5225 0    50   ~ 0
 <- ENABLE 3V3_USB
@@
 Text Notes 6375 5025 0    50   ~ 0
 PWR_OUT -->
+Wire Wire Line
+	9350 5025 6050 5025
 $EndSCHEMATC
