File: STM32MP1_TestBoard/Power_MPU.sch (KiCad schematic (older format))
At the start: 30 parts, among them U1 STM32MP157xAB

Commit message: updated schematic
changed STM32MP157xAB to STM32MP157xAC
Parts:
- U1: value STM32MP157xAB -> STM32MP157xAC
Changed lines of the file:
@@
 P 8175 4425
 F 0 "U1" H 8175 6340 50  0000 C CNN
-F 1 "STM32MP157xAB" H 8175 6249 50  0000 C CNN
+F 1 "STM32MP157xAC" H 8175 6249 50  0000 C CNN
 F 2 "STM32MP151_LFBGA:BGA-361_19x19_16.0x16.0mm" H 8025 6325 50  0001 C CNN
 F 3 "https://www.st.com/resource/en/datasheet/stm32mp151c.pdf" H 8825 4575 50  0001 C CNN

Commit message: corrected STM32MP157 footprint
Parts:
- U1: value STM32MP157xAC -> STM32MP157xAB; footprint STM32MP151_LFBGA:BGA-361_19x19_16.0x16.0mm -> STM32MP151_LFBGA:BGA-354_19x19_16.0x16.0mm
Changed lines of the file:
@@
 P 8175 4425
 F 0 "U1" H 8175 6340 50  0000 C CNN
-F 1 "STM32MP157xAC" H 8175 6249 50  0000 C CNN
-F 2 "STM32MP151_LFBGA:BGA-361_19x19_16.0x16.0mm" H 8025 6325 50  0001 C CNN
+F 1 "STM32MP157xAB" H 8175 6249 50  0000 C CNN
+F 2 "STM32MP151_LFBGA:BGA-354_19x19_16.0x16.0mm" H 8025 6325 50  0001 C CNN
 F 3 "https://www.st.com/resource/en/datasheet/stm32mp151c.pdf" H 8825 4575 50  0001 C CNN
 F 4 "~" H 8175 4425 50  0001 C CNN "Mfr"
