File: STM32MP1_TestBoard/GPIO.sch (KiCad schematic (older format))
At the start: 16 parts, among them J10 Conn_01x16, J11 Conn_01x16, J3 Conn_02x03_Odd_Even, J4 Conn_01x16, J5 Conn_01x06, J6 Conn_01x16, J7 Conn_01x16, J8 Conn_01x12, J9 Conn_01x06, U1 STM32MP157xAB

Commit message: layout update
backup. work in progress
Changed lines of the file:
@@
 Text Label 10300 2200 0    50   ~ 0
 SDMMC1_D0
-Text Label 4500 1975 2    50   ~ 0
+Text Label 4500 2025 2    50   ~ 0
 SDMMC1_D0
 Wire Wire Line
-	3675 1975 4500 1975
-Wire Wire Line
-	3675 2075 4500 2075
-Text Label 4500 2075 2    50   ~ 0
+	3675 2025 4500 2025
+Wire Wire Line
+	3675 2125 4500 2125
+Text Label 4500 2125 2    50   ~ 0
 SDMMC1_D1
 Wire Wire Line
-	3675 2175 4500 2175
-Text Label 4500 2175 2    50   ~ 0
+	3675 2225 4500 2225
+Text Label 4500 2225 2    50   ~ 0
 SDMMC1_D2
 Wire Wire Line
-	3675 2275 4500 2275
-Text Label 4500 2275 2    50   ~ 0
+	3675 2325 4500 2325
+Text Label 4500 2325 2    50   ~ 0
 SDMMC1_D3
 Text Label 10300 2300 0    50   ~ 0
@@
 F0 "USB_Conn" 50
 F1 "USB_Conn.sch" 50
-F2 "USBC_DM" I R 3825 5000 50
-F3 "USBC_DP" I R 3825 5100 50
-F4 "USBA_DP" I R 3825 5300 50
-F5 "USBA_DM" I R 3825 5200 50
+F2 "USB_D1_P" I R 3825 5100 50
+F3 "USB_D2_P" I R 3825 5300 50
+F4 "USB_D1_N" I R 3825 5000 50
+F5 "USB_D2_N" I R 3825 5200 50
 $EndSheet
 Wire Wire Line
@@
 F8 "3V3_SDIO_VDD" I R 3675 2925 50
 $EndSheet
-Text Label 4500 3375 2    50   ~ 0
-SDMMC1_D0
-Wire Wire Line
-	3675 3375 4500 3375
-Wire Wire Line
-	3675 3475 4500 3475
-Text Label 4500 3475 2    50   ~ 0
-SDMMC1_D1
-Wire Wire Line
-	3675 3575 4500 3575
-Text Label 4500 3575 2    50   ~ 0
-SDMMC1_D2
-Wire Wire Line
-	3675 3675 4500 3675
-Text Label 4500 3675 2    50   ~ 0
-SDMMC1_D3
+Text Label 4500 3425 2    50   ~ 0
+SDMMC2_D0
+Wire Wire Line
+	3675 3425 4500 3425
+Wire Wire Line
+	3675 3525 4500 3525
+Text Label 4500 3525 2    50   ~ 0
+SDMMC2_D1
+Wire Wire Line
+	3675 3625 4500 3625
+Text Label 4500 3625 2    50   ~ 0
+SDMMC2_D2
+Wire Wire Line
+	3675 3725 4500 3725
+Text Label 4500 3725 2    50   ~ 0
+SDMMC2_D3
 Text Label 4500 3200 2    50   ~ 0
-SDMMC1_CMD
+SDMMC2_CMD
 Wire Wire Line
 	4500 3200 3675 3200
@@
 	3675 3100 4500 3100
 Text Label 4500 3100 2    50   ~ 0
-SDMMC1_CK
+SDMMC2_CK
 Text HLabel 3950 2925 2    50   Input ~ 0
 3V3_SDIO_VDD

Commit message: updated to use stm32MP15x symbol library
Parts:
- U1: Mfr STMicroelectronics -> (none); PartNo STM32MP157FAB -> (none)
Changed lines of the file:
@@
 	8025 5300 3825 5300
-$Comp
-L STM32MP15x:STM32MP157xAB U?
-U 1 1 609989B0
-P 8875 3300
-AR Path="/609989B0" Ref="U?"  Part="1"
-AR Path="/6097C138/609989B0" Ref="U1"  Part="1"
-F 0 "U1" H 8925 5465 50  0000 C CNN
-F 1 "STM32MP157xAB" H 8925 5374 50  0000 C CNN
-F 2 "STM32MP151_LFBGA:BGA-361_19x19_16.0x16.0mm" H 8725 5200 50  0001 C CNN
-F 3 "https://www.st.com/resource/en/datasheet/stm32mp157f.pdf" H 9175 3800 50  0001 C CNN
-F 4 "STMicroelectronics" H 8875 3300 50  0001 C CNN "Mfr"
-F 5 "STM32MP157FAB" H 8875 3300 50  0001 C CNN "PartNo"
-	1    8875 3300
-	1    0    0    -1
-$EndComp
-$Comp
-L STM32MP15x:STM32MP157xAB U?
-U 2 1 609989B8
-P 8900 8225
-AR Path="/609989B8" Ref="U?"  Part="2"
-AR Path="/6097C138/609989B8" Ref="U1"  Part="2"
-F 0 "U1" H 8900 9790 50  0000 C CNN
-F 1 "STM32MP157xAB" H 8900 9699 50  0000 C CNN
-F 2 "STM32MP151_LFBGA:BGA-361_19x19_16.0x16.0mm" H 8750 10125 50  0001 C CNN
-F 3 "https://www.st.com/resource/en/datasheet/stm32mp157f.pdf" H 9200 8725 50  0001 C CNN
-F 4 "STMicroelectronics" H 8900 8225 50  0001 C CNN "Mfr"
-F 5 "STM32MP157FAB" H 8900 8225 50  0001 C CNN "PartNo"
-	2    8900 8225
-	1    0    0    -1
-$EndComp
 $Comp
 L Connector_Generic:Conn_01x06 J?
@@
 Wire Wire Line
 	14275 8100 14525 8100
+$Comp
+L STM32MP15x:STM32MP157xAB U1
+U 2 1 5FC247C4
+P 8900 8225
+F 0 "U1" H 8900 9790 50  0000 C CNN
+F 1 "STM32MP157xAB" H 8900 9699 50  0000 C CNN
+F 2 "STM32MP151_LFBGA:BGA-361_19x19_16.0x16.0mm" H 8750 10125 50  0001 C CNN
+F 3 "https://www.st.com/resource/en/datasheet/stm32mp151c.pdf" H 9550 8375 50  0001 C CNN
+	2    8900 8225
+	1    0    0    -1
+$EndComp
+$Comp
+L STM32MP15x:STM32MP157xAB U1
+U 1 1 5FC44781
+P 8875 3300
+F 0 "U1" H 8925 5465 50  0000 C CNN
+F 1 "STM32MP157xAB" H 8925 5374 50  0000 C CNN
+F 2 "STM32MP151_LFBGA:BGA-361_19x19_16.0x16.0mm" H 8725 5200 50  0001 C CNN
+F 3 "https://www.st.com/resource/en/datasheet/stm32mp151c.pdf" H 9525 3450 50  0001 C CNN
+	1    8875 3300
+	1    0    0    -1
+$EndComp
 $EndSCHEMATC

Commit message: added traces for sdio, dsi and swd connectors
Parts:
- removed J10, J11, J4, J6, J7: Conn_01x16, Connector_PinHeader_2.54mm:PinHeader_1x16_P2.54mm_Vertical, symbol Connector_Generic:Conn_01x16
- removed J5, J9: Conn_01x06, Connector_PinHeader_2.54mm:PinHeader_1x06_P2.54mm_Vertical, symbol Connector_Generic:Conn_01x06
- removed J8: Conn_01x12, Connector_PinHeader_2.54mm:PinHeader_1x12_P2.54mm_Vertical, symbol Connector_Generic:Conn_01x12
- added J1, J2, J3, J4: Conn_01x27, Connector_PinHeader_2.54mm:PinHeader_1x27_P2.54mm_Vertical, symbol Connector_Generic:Conn_01x27
- added J7: Conn_01x06, Connector_PinHeader_2.54mm:PinHeader_1x06_P2.54mm_Vertical, symbol Connector_Generic:Conn_01x06
- renumbered J3 to J5
Connections:
- net BOOT_STATUS: now also J1.13 (Pin_13)
- net DSI_D0_N: now reaches U1.A13 (DSI_D0_N)
- net DSI_D0_N: now also J7.6 (Pin_6)
- net DSI_CK_N: now reaches U1.A14 (DSI_CK_N)
- net DSI_CK_N: now also J7.4 (Pin_4)
- net DSI_D1_N: now reaches U1.A15 (DSI_D1_N)
- net DSI_D1_N: now also J7.2 (Pin_2)
- net PG15: now reaches U1.A2 (PG15)
- net PG15: now also J4.17 (Pin_17)
- net PE3: now reaches U1.A5 (PE3)
- net PE3: now also J4.19 (Pin_19)
- net PG6: now reaches U1.A6 (PG6)
- net PG6: now also J3.20 (Pin_20)
- net PE1: now reaches U1.B1 (PE1)
- net PE1: now also J3.17 (Pin_17)
- net PE4: now reaches U1.B11 (PE4)
- net PE4: now also J1.25 (Pin_25)
- net DSI_D0_P: now reaches U1.B13 (DSI_D0_P)
- net DSI_D0_P: now also J7.5 (Pin_5)
- net DSI_CK_P: now reaches U1.B14 (DSI_CK_P)
- net DSI_CK_P: now also J7.3 (Pin_3)
- net DSI_D1_P: now reaches U1.B15 (DSI_D1_P)
- net DSI_D1_P: now also J7.1 (Pin_1)
- net PE6: now reaches U1.B3 (PE6)
- net PE6: now also J1.18 (Pin_18)
- net PE5: now reaches U1.B7 (PE5)
- net PE5: now also J2.21 (Pin_21)
- net PE11: now reaches U1.C1 (PE11)
- net PE11: now also J1.17 (Pin_17)
- net PE13: now reaches U1.C2 (PE13)
- net PE13: now also J2.17 (Pin_17)
- net PE0: now reaches U1.C4 (PE0)
- net PE0: now also J3.18 (Pin_18)
- net PE12: now reaches U1.D2 (PE12)
- net PE12: now also J3.16 (Pin_16)
- net PE14: now reaches U1.D3 (PE14)
- net PE14: now also J4.16 (Pin_16)
- net PE15: now reaches U1.E1 (PE15)
- net PE15: now also J2.16 (Pin_16)
- net PG12: now reaches U1.F1 (PG12)
- net PG12: now also J4.15 (Pin_15)
- net PH0: now reaches U1.M1 (PH0-OSC_IN)
- net PH0: now also J3.13 (Pin_13)
- net PH1: now reaches U1.M2 (PH1-OSC_OUT)
- net PH1: now also J2.13 (Pin_13)
- net PE2: now reaches U1.T1 (PE2)
- net PE2: now also J4.11 (Pin_11)
- net PE7: now reaches U1.T10 (PE7)
- net PE7: now also J4.3 (Pin_3)
- net PE8: now reaches U1.T11 (PE8)
- net PE8: now also J4.2 (Pin_2)
- net PG9: now reaches U1.T14 (PG9)
- net PG9: now also J4.1 (Pin_1)
- net PG14: now reaches U1.U1 (PG14)
- net PG14: now also J1.11 (Pin_11)
- net PF8: now reaches U1.U10 (PF8)
- net PF8: now also J1.4 (Pin_4)
- net PG13: now reaches U1.U2 (PG13)
- net PG13: now also J4.10 (Pin_10)
- net PF11: now reaches U1.U5 (PF11)
- net PF11: now also J4.7 (Pin_7)
- net PG8: now reaches U1.U7 (PG8)
- net PG8: now also J3.6 (Pin_6)
- net PF10: now reaches U1.U9 (PF10)
- net PF10: now also J3.5 (Pin_5)
- net PE10: now reaches U1.V10 (PE10)
- net PE10: now also J3.3 (Pin_3)
- net PG11: now reaches U1.V6 (PG11)
- net PG11: now also J2.7 (Pin_7)
- net PG10: now reaches U1.V7 (PG10)
- net PG10: now also J2.6 (Pin_6)
- net PF6: now reaches U1.V9 (PF6)
- net PF6: now also J3.4 (Pin_4)
- net PG7: now reaches U1.W10 (PG7)
- net PG7: now also J2.3 (Pin_3)
- net PE9: now reaches U1.W7 (PE9)
- net PE9: now also J1.6 (Pin_6)
- net PF7: now reaches U1.W8 (PF7)
- net PF7: now also J1.5 (Pin_5)
- net PF9: now reaches U1.W9 (PF9)
- net PF9: now also J2.4 (Pin_4)
- net PD0: now reaches U1.A3 (PD0)
- net PD0: now also J2.18 (Pin_18)
- net PD1: now reaches U1.A4 (PD1)
- net PD1: now also J1.19 (Pin_19)
- net PC7: now reaches U1.A9 (PC7)
- net PC7: now also J2.23 (Pin_23)
- net PD7: now reaches U1.B4 (PD7)
- net PD7: now also J4.18 (Pin_18)
- net PB7: now reaches U1.B5 (PB7)
- net PB7: now also J3.19 (Pin_19)
- net PA8: now reaches U1.B8 (PA8)
- net PA8: now also J1.22 (Pin_22)
- net PD10: now reaches U1.C5 (PD10)
- net PD10: now also J2.19 (Pin_19)
- net PD3: now reaches U1.C6 (PD3)
- net PD3: now also J2.20 (Pin_20)
- net PA15: now reaches U1.C7 (PA15)
- net PA15: now also J1.21 (Pin_21)
- net PA9: now reaches U1.C8 (PA9)
- net PA9: now also J4.21 (Pin_21)
- net PB14: now reaches U1.C9 (PB14)
- net PB14: now also J4.22 (Pin_22)
- net PC6: now reaches U1.D10 (PC6)
- net PC6: now also J3.23 (Pin_23)
- net PD4: now reaches U1.D6 (PD4)
- net PD4: now also J1.20 (Pin_20)
- net PD5: now reaches U1.D7 (PD5)
- net PD5: now also J4.20 (Pin_20)
- net PB9: now reaches U1.D9 (PB9)
- net PB9: now also J3.22 (Pin_22)
- net PD6: now reaches U1.E3 (PD6)
- net PD6: now also J1.16 (Pin_16)
- net PD8: now reaches U1.F2 (PD8)
- net PD8: now also J3.15 (Pin_15)
- net PD14: now reaches U1.F3 (PD14)
- net PD14: now also J2.15 (Pin_15)
- net PD15: now reaches U1.G1 (PD15)
- net PD15: now also J1.15 (Pin_15)
- net PD9: now reaches U1.G3 (PD9)
- net PD9: now also J4.14 (Pin_14)
- net PC14: now reaches U1.H1 (PC14-OSC32_IN)
- net PC14: now also J3.14 (Pin_14)
- net PC15: now reaches U1.H2 (PC15-OSC32_OUT)
- net PC15: now also J2.14 (Pin_14)
- net PC13: now reaches U1.K3 (PC13)
- net PC13: now also J1.14 (Pin_14)
- net PA3: now reaches U1.P3 (PA3)
- net PA3: now also J4.13 (Pin_13)
- net PA5: now reaches U1.P4 (PA5)
- net PA5: now also J4.12 (Pin_12)
- net PA14: now reaches U1.R1 (PA14)
- net PA14: now also J3.12 (Pin_12)
- net PA4: now reaches U1.R4 (PA4)
- net PA4: now also J1.12 (Pin_12)
- net PB6: now reaches U1.T12 (PB6)
- net PB6: now also J2.2 (Pin_2)
- net PB2: now reaches U1.T13 (PB2)
- net PB2: now also J1.2 (Pin_2)
- net PA10: now reaches U1.T16 (PA10)
- net PA10: now also J3.1 (Pin_1)
- net PC2: now reaches U1.T2 (PC2)
- net PC2: now also J3.11 (Pin_11)
- net PC3: now reaches U1.T3 (PC3)
- net PC3: now also J2.11 (Pin_11)
- net PA6: now reaches U1.T5 (PA6)
- net PA6: now also J3.8 (Pin_8)
- net PA7: now reaches U1.T6 (PA7)
- net PA7: now also J3.7 (Pin_7)
- net PC0: now reaches U1.T7 (PC0)
- net PC0: now also J4.6 (Pin_6)
- net PB5: now reaches U1.T8 (PB5)
- net PB5: now also J4.5 (Pin_5)
- net PD12: now reaches U1.U11 (PD12)
- net PD12: now also J1.3 (Pin_3)
- net PD13: now reaches U1.U12 (PD13)
- net PD13: now also J3.2 (Pin_2)
- net PA12: now reaches U1.U16 (PA12)
- net PA12: now also J2.1 (Pin_1)
- net PA1: now reaches U1.U4 (PA1)
- net PA1: now also J4.8 (Pin_8)
- net PB11: now reaches U1.V1 (PB11)
- net PB11: now also J3.10 (Pin_10)
- net PA11: now reaches U1.V17 (PA11)
- net PA11: now also J1.1 (Pin_1)
- net PB1: now reaches U1.V3 (PB1)
- net PB1: now also J4.9 (Pin_9)
- net PC5: now reaches U1.V4 (PC5)
- net PC5: now also J2.9 (Pin_9)
- net PB12: now reaches U1.V5 (PB12)
- net PB12: now also J2.8 (Pin_8)
- net PD11: now reaches U1.V8 (PD11)
- net PD11: now also J2.5 (Pin_5)
- net PA2: now reaches U1.W2 (PA2)
- net PA2: now also J1.10 (Pin_10)
- net PB0: now reaches U1.W3 (PB0)
- net PB0: now also J3.9 (Pin_9)
- net PC4: now reaches U1.W4 (PC4)
- net PC4: now also J1.9 (Pin_9)
- net PB10: now reaches U1.W5 (PB10)
- net PB10: now also J1.8 (Pin_8)
- net PB8: now reaches U1.W6 (PB8)
- net PB8: now also J1.7 (Pin_7)
- net SDMMC1_CK renamed PC12
- net PC12: now also J4.23 (Pin_23)
- net SDMMC1_CMD renamed PD2
- net PD2: now also J1.24 (Pin_24)
- net SDMMC1_D0 renamed PC8
- net PC8: now also J4.24 (Pin_24)
- net SDMMC1_D1 renamed PC9
- net PC9: now also J2.24 (Pin_24)
- net SDMMC1_D2 renamed PC10
- net PC10: now also J3.24 (Pin_24)
- net SDMMC1_D3 renamed PC11
- net PC11: now also J2.25 (Pin_25)
- net SDMMC2_CK renamed PC1
- net PC1: now also J2.10 (Pin_10)
- net SDMMC2_CMD renamed PA0
- net PA0: now also J2.12 (Pin_12)
- net SDMMC2_D0 renamed PB13
- net PB13: now also J4.4 (Pin_4)
- net SDMMC2_D1 renamed PB15
- net PB15: now also J2.22 (Pin_22)
- net SDMMC2_D2 renamed PB3
- net PB3: now also J3.21 (Pin_21)
- net SDMMC2_D3 renamed PB4
- net PB4: now also J1.23 (Pin_23)
- no-connect marks 1 -> 11
Other:
- moved on the sheet: D1, R9

Commit message: updated RevA draft
- added silkscreen
Parts:
- removed J7: Conn_01x06, Connector_PinHeader_2.54mm:PinHeader_1x06_P2.54mm_Vertical, symbol Connector_Generic:Conn_01x06
- added J7: Conn_01x08, Connector_PinHeader_2.54mm:PinHeader_1x08_P2.54mm_Vertical, symbol Connector_Generic:Conn_01x08
Connections:
- net 3.3V_VDD: now also J1.26 (Pin_26), J2.26 (Pin_26), J3.26 (Pin_26), J4.26 (Pin_26), J7.1 (Pin_1)
- net DSI_CK_N: now also J7.6 (Pin_6)
- net DSI_CK_P: now also J7.5 (Pin_5)
- net DSI_D0_N: now also J7.8 (Pin_8)
- net DSI_D0_P: now also J7.7 (Pin_7)
- net DSI_D1_N: now also J7.4 (Pin_4)
- net DSI_D1_P: now also J7.3 (Pin_3)
- net GNDS: now also J1.27 (Pin_27), J2.27 (Pin_27), J3.27 (Pin_27), J4.27 (Pin_27), J7.2 (Pin_2)
- no-connect marks 11 -> 3
Changed lines of the file:
@@
 Text Label 14000 7600 2    50   ~ 0
 PC11
-$Comp
-L Connector_Generic:Conn_01x27 J1
-U 1 1 6094EFEE
-P 15775 2800
-F 0 "J1" H 15855 2842 50  0000 L CNN
-F 1 "Conn_01x27" H 15855 2751 50  0000 L CNN
-F 2 "Connector_PinHeader_2.54mm:PinHeader_1x27_P2.54mm_Vertical" H 15775 2800 50  0001 C CNN
-F 3 "~" H 15775 2800 50  0001 C CNN
-	1    15775 2800
-	1    0    0    -1
-$EndComp
-$Comp
-L Connector_Generic:Conn_01x27 J2
-U 1 1 6095B1D0
-P 15775 6500
-F 0 "J2" H 15855 6542 50  0000 L CNN
-F 1 "Conn_01x27" H 15855 6451 50  0000 L CNN
-F 2 "Connector_PinHeader_2.54mm:PinHeader_1x27_P2.54mm_Vertical" H 15775 6500 50  0001 C CNN
-F 3 "~" H 15775 6500 50  0001 C CNN
-	1    15775 6500
-	1    0    0    -1
-$EndComp
-$Comp
-L Connector_Generic:Conn_01x27 J3
-U 1 1 609704E3
-P 19775 2800
-F 0 "J3" H 19855 2842 50  0000 L CNN
-F 1 "Conn_01x27" H 19855 2751 50  0000 L CNN
-F 2 "Connector_PinHeader_2.54mm:PinHeader_1x27_P2.54mm_Vertical" H 19775 2800 50  0001 C CNN
-F 3 "~" H 19775 2800 50  0001 C CNN
-	1    19775 2800
-	1    0    0    -1
-$EndComp
-$Comp
-L Connector_Generic:Conn_01x27 J4
-U 1 1 60976149
-P 19775 6500
-F 0 "J4" H 19855 6542 50  0000 L CNN
-F 1 "Conn_01x27" H 19855 6451 50  0000 L CNN
-F 2 "Connector_PinHeader_2.54mm:PinHeader_1x27_P2.54mm_Vertical" H 19775 6500 50  0001 C CNN
-F 3 "~" H 19775 6500 50  0001 C CNN
-	1    19775 6500
-	1    0    0    -1
-$EndComp
-NoConn ~ 19575 7800
-NoConn ~ 19575 4100
 Wire Wire Line
 	19575 5300 18000 5300
@@
 Text Label 18000 3000 2    50   ~ 0
 PE12
-NoConn ~ 15575 7700
-NoConn ~ 15575 7800
-NoConn ~ 19575 7600
-NoConn ~ 19575 7700
-NoConn ~ 19575 3900
-NoConn ~ 19575 4000
-NoConn ~ 15575 4000
-NoConn ~ 15575 4100
+Wire Wire Line
+	9800 8225 11800 8225
+Wire Wire Line
+	9800 8325 11800 8325
+Wire Wire Line
+	9800 8425 11800 8425
+Wire Wire Line
+	9800 8525 11800 8525
+Wire Wire Line
+	9800 8625 11800 8625
+Wire Wire Line
+	9800 8725 11800 8725
 $Comp
-L Connector_Generic:Conn_01x06 J7
-U 1 1 622AE579
-P 11600 8425
-F 0 "J7" H 11680 8417 50  0000 L CNN
-F 1 "Conn_01x06" H 11680 8326 50  0000 L CNN
-F 2 "Connector_PinHeader_2.54mm:PinHeader_1x06_P2.54mm_Vertical" H 11600 8425 50  0001 C CNN
-F 3 "~" H 11600 8425 50  0001 C CNN
-	1    11600 8425
+L Connector_Generic:Conn_01x27 J1
+U 1 1 6094EFEE
+P 15775 2800
+F 0 "J1" H 15855 2842 50  0000 L CNN
+F 1 "Conn_01x27" H 15855 2751 50  0000 L CNN
+F 2 "Connector_PinHeader_2.54mm:PinHeader_1x27_P2.54mm_Vertical" H 15775 2800 50  0001 C CNN
+F 3 "~" H 15775 2800 50  0001 C CNN
+	1    15775 2800
+	1    0    0    -1
+$EndComp
+$Comp
+L Connector_Generic:Conn_01x27 J3
+U 1 1 609704E3
+P 19775 2800
+F 0 "J3" H 19855 2842 50  0000 L CNN
+F 1 "Conn_01x27" H 19855 2751 50  0000 L CNN
+F 2 "Connector_PinHeader_2.54mm:PinHeader_1x27_P2.54mm_Vertical" H 19775 2800 50  0001 C CNN
+F 3 "~" H 19775 2800 50  0001 C CNN
+	1    19775 2800
+	1    0    0    -1
+$EndComp
+$Comp
+L Connector_Generic:Conn_01x27 J4
+U 1 1 60976149
+P 19775 6500
+F 0 "J4" H 19855 6542 50  0000 L CNN
+F 1 "Conn_01x27" H 19855 6451 50  0000 L CNN
+F 2 "Connector_PinHeader_2.54mm:PinHeader_1x27_P2.54mm_Vertical" H 19775 6500 50  0001 C CNN
+F 3 "~" H 19775 6500 50  0001 C CNN
+	1    19775 6500
+	1    0    0    -1
+$EndComp
+$Comp
+L Connector_Generic:Conn_01x27 J2
+U 1 1 6095B1D0
+P 15775 6500
+F 0 "J2" H 15855 6542 50  0000 L CNN
+F 1 "Conn_01x27" H 15855 6451 50  0000 L CNN
+F 2 "Connector_PinHeader_2.54mm:PinHeader_1x27_P2.54mm_Vertical" H 15775 6500 50  0001 C CNN
+F 3 "~" H 15775 6500 50  0001 C CNN
+	1    15775 6500
 	1    0    0    -1
 $EndComp
 Wire Wire Line
-	9800 8225 11400 8225
+	15575 4100 15125 4100
 Wire Wire Line
-	9800 8325 11400 8325
+	15125 4100 15125 4375
+$Comp
+L power:GNDS #PWR0103
+U 1 1 60195BDC
+P 15125 4375
+F 0 "#PWR0103" H 15125 4125 50  0001 C CNN
+F 1 "GNDS" H 15130 4202 50  0000 C CNN
+F 2 "" H 15125 4375 50  0001 C CNN
+F 3 "" H 15125 4375 50  0001 C CNN
+	1    15125 4375
+	1    0    0    -1
+$EndComp
 Wire Wire Line
-	9800 8425 11400 8425
+	19575 4100 19125 4100
 Wire Wire Line
-	9800 8525 11400 8525
+	19125 4100 19125 4375
+$Comp
+L power:GNDS #PWR0104
+U 1 1 60196142
+P 19125 4375
+F 0 "#PWR0104" H 19125 4125 50  0001 C CNN
+F 1 "GNDS" H 19130 4202 50  0000 C CNN
+F 2 "" H 19125 4375 50  0001 C CNN
+F 3 "" H 19125 4375 50  0001 C CNN
+	1    19125 4375
+	1    0    0    -1
+$EndComp
 Wire Wire Line
-	9800 8625 11400 8625
+	19575 7800 19125 7800
 Wire Wire Line
-	9800 8725 11400 8725
+	19125 7800 19125 8075
+$Comp
+L power:GNDS #PWR0105
+U 1 1 601B0472
+P 19125 8075
+F 0 "#PWR0105" H 19125 7825 50  0001 C CNN
+F 1 "GNDS" H 19130 7902 50  0000 C CNN
+F 2 "" H 19125 8075 50  0001 C CNN
+F 3 "" H 19125 8075 50  0001 C CNN
+	1    19125 8075
+	1    0    0    -1
+$EndComp
+Wire Wire Line
+	15575 7800 15125 7800
+Wire Wire Line
+	15125 7800 15125 8075
+$Comp
+L power:GNDS #PWR0106
+U 1 1 601E5077
+P 15125 8075
+F 0 "#PWR0106" H 15125 7825 50  0001 C CNN
+F 1 "GNDS" H 15130 7902 50  0000 C CNN
+F 2 "" H 15125 8075 50  0001 C CNN
+F 3 "" H 15125 8075 50  0001 C CNN
+	1    15125 8075
+	1    0    0    -1
+$EndComp
+Text HLabel 19200 7700 0    50   Input ~ 0
+3.3V_VDD
+Wire Wire Line
+	19575 7700 19200 7700
+Text HLabel 15200 7700 0    50   Input ~ 0
+3.3V_VDD
+Wire Wire Line
+	15575 7700 15200 7700
+Text HLabel 15200 4000 0    50   Input ~ 0
+3.3V_VDD
+Wire Wire Line
+	15575 4000 15200 4000
+Text HLabel 19200 4000 0    50   Input ~ 0
+3.3V_VDD
+Wire Wire Line
+	19575 4000 19200 4000
+NoConn ~ 19575 7600
+NoConn ~ 19575 3900
+$Comp
+L Connector_Generic:Conn_01x08 J7
+U 1 1 603AE8E8
+P 12000 8325
+F 0 "J7" H 12080 8317 50  0000 L CNN
+F 1 "Conn_01x08" H 12080 8226 50  0000 L CNN
+F 2 "Connector_PinHeader_2.54mm:PinHeader_1x08_P2.54mm_Vertical" H 12000 8325 50  0001 C CNN
+F 3 "~" H 12000 8325 50  0001 C CNN
+	1    12000 8325
+	1    0    0    -1
+$EndComp
+Wire Wire Line
+	11800 8025 11650 8025
+Wire Wire Line
+	11650 8025 11650 7700
+Text HLabel 11650 7700 1    50   Input ~ 0
+3.3V_VDD
+Wire Wire Line
+	11800 8125 11500 8125
+$Comp
+L power:GNDS #PWR08
+U 1 1 60456FA5
+P 11500 8125
+F 0 "#PWR08" H 11500 7875 50  0001 C CNN
+F 1 "GNDS" V 11505 7997 50  0000 R CNN
+F 2 "" H 11500 8125 50  0001 C CNN
+F 3 "" H 11500 8125 50  0001 C CNN
+	1    11500 8125
+	0    1    1    0
+$EndComp
 $EndSCHEMATC

Commit message: RevA layout final
Parts:
- R9: value 680R -> 1K
Changed lines of the file:
@@
 AR Path="/6097C138/609989E7" Ref="R9"  Part="1"
 F 0 "R9" V 9100 10750 50  0000 C CNN
-F 1 "680R" V 8900 10750 50  0000 C CNN
+F 1 "1K" V 8900 10750 50  0000 C CNN
 F 2 "Resistor_SMD:R_0402_1005Metric_Pad0.72x0.64mm_HandSolder" V 8930 10750 50  0001 C CNN
 F 3 "~" H 9000 10750 50  0001 C CNN

Commit message: updated schema and bom docs
Parts:
- U1: value STM32MP157xAB -> STM32MP157xAC
Changed lines of the file:
@@
 F 2 "LED_SMD:LED_0805_2012Metric_Pad1.15x1.40mm_HandSolder" H 9400 10425 50  0001 C CNN
 F 3 "~" H 9400 10425 50  0001 C CNN
+F 4 "~" H 9400 10425 50  0001 C CNN "Mfr"
+F 5 "~" H 9400 10425 50  0001 C CNN "PartNo"
 	1    9400 10425
 	0    -1   -1   0
@@
 P 8900 8225
 F 0 "U1" H 8900 9790 50  0000 C CNN
-F 1 "STM32MP157xAB" H 8900 9699 50  0000 C CNN
+F 1 "STM32MP157xAC" H 8900 9699 50  0000 C CNN
 F 2 "STM32MP151_LFBGA:BGA-361_19x19_16.0x16.0mm" H 8750 10125 50  0001 C CNN
 F 3 "https://www.st.com/resource/en/datasheet/stm32mp151c.pdf" H 9550 8375 50  0001 C CNN
+F 4 "~" H 8900 8225 50  0001 C CNN "Mfr"
+F 5 "~" H 8900 8225 50  0001 C CNN "PartNo"
 	2    8900 8225
 	1    0    0    -1
@@
 P 8875 3300
 F 0 "U1" H 8925 5465 50  0000 C CNN
-F 1 "STM32MP157xAB" H 8925 5374 50  0000 C CNN
+F 1 "STM32MP157xAC" H 8925 5374 50  0000 C CNN
 F 2 "STM32MP151_LFBGA:BGA-361_19x19_16.0x16.0mm" H 8725 5200 50  0001 C CNN
 F 3 "https://www.st.com/resource/en/datasheet/stm32mp151c.pdf" H 9525 3450 50  0001 C CNN
+F 4 "~" H 8875 3300 50  0001 C CNN "Mfr"
+F 5 "~" H 8875 3300 50  0001 C CNN "PartNo"
 	1    8875 3300
 	1    0    0    -1
@@
 F 2 "Connector_PinHeader_2.54mm:PinHeader_1x27_P2.54mm_Vertical" H 15775 2800 50  0001 C CNN
 F 3 "~" H 15775 2800 50  0001 C CNN
+F 4 "~" H 15775 2800 50  0001 C CNN "Mfr"
+F 5 "~" H 15775 2800 50  0001 C CNN "PartNo"
 	1    15775 2800
 	1    0    0    -1
@@
 F 2 "Connector_PinHeader_2.54mm:PinHeader_1x27_P2.54mm_Vertical" H 19775 2800 50  0001 C CNN
 F 3 "~" H 19775 2800 50  0001 C CNN
+F 4 "~" H 19775 2800 50  0001 C CNN "Mfr"
+F 5 "~" H 19775 2800 50  0001 C CNN "PartNo"
 	1    19775 2800
 	1    0    0    -1
@@
 F 2 "Connector_PinHeader_2.54mm:PinHeader_1x27_P2.54mm_Vertical" H 19775 6500 50  0001 C CNN
 F 3 "~" H 19775 6500 50  0001 C CNN
+F 4 "~" H 19775 6500 50  0001 C CNN "Mfr"
+F 5 "~" H 19775 6500 50  0001 C CNN "PartNo"
 	1    19775 6500
 	1    0    0    -1
@@
 F 2 "Connector_PinHeader_2.54mm:PinHeader_1x27_P2.54mm_Vertical" H 15775 6500 50  0001 C CNN
 F 3 "~" H 15775 6500 50  0001 C CNN
+F 4 "~" H 15775 6500 50  0001 C CNN "Mfr"
+F 5 "~" H 15775 6500 50  0001 C CNN "PartNo"
 	1    15775 6500
 	1    0    0    -1
@@
 F 2 "Connector_PinHeader_2.54mm:PinHeader_1x08_P2.54mm_Vertical" H 12000 8325 50  0001 C CNN
 F 3 "~" H 12000 8325 50  0001 C CNN
+F 4 "~" H 12000 8325 50  0001 C CNN "Mfr"
+F 5 "~" H 12000 8325 50  0001 C CNN "PartNo"
 	1    12000 8325
 	1    0    0    -1
